File: KICAD PCBs/BackPCB-Acrylic/BackPCB-Acry.kicad_pcb (KiCad board)
At the start: 2 copper layers, 347 x 156.3 mm, 19 parts

Commit message: modified switch plate and backplate
Parts:
- removed the H0 at (41.2, 63.4)
- removed the H1 at (377.8, 62.7)
- removed the H10 at (376.0, 116.0)
- removed the H3 at (40.1, 196.3)
- removed the H6 at (212.2, 116.0)
- removed the H9 at (48.3, 116.0)
- moved H1 2.12 mm to (379.8, 63.4)
- moved H7 1.30 mm to (203.8, 177.3)
- moved H3 0.71 mm to (40.2, 197.0)
- moved H11 0.35 mm to (182.9, 63.8)
- moved H4 0.05 mm to (325.2, 209.8)
Other:
- board text removed: "<Stepped NotStepped>"
Changed lines of the file:
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@@
   (net 0 "")
   (footprint "MountingHole:MountingHole_2.2mm_M2_Pad" (layer "F.Cu")
-    (at 376 116)
-    (descr "Mounting Hole 2.2mm, M2")
-    (tags "mounting hole 2.2mm m2")
-    (property "Sheetfile" "BackPCB-Acry.kicad_sch")
-    (property "Sheetname" "")
-    (attr exclude_from_pos_files)
-    (fp_text reference "H10" (at 0 -3.2) (layer "Dwgs.User")
-      (effects (font (size 1 1) (thickness 0.15)))
-    )
-    (fp_text value "MountingHole" (at 0 3.2) (layer "F.Fab")
-      (effects (font (size 1 1) (thickness 0.15)))
-    )
-    (fp_text user "${REFERENCE}" (at 0.3 0) (layer "F.Fab")
-      (effects (font (size 1 1) (thickness 0.15)))
-    )
-    (fp_circle (center 0 0) (end 2.2 0) (layer "Cmts.User") (width 0.1) (fill none))
-    (fp_circle (center 0 0) (end 2.45 0) (layer "F.CrtYd") (width 0.1) (fill none))
-    (pad "1" thru_hole circle locked (at 0 0) (size 4.4 4.4) (drill 2.2) (layers *.Cu *.Mask))
-  )
-  (footprint "MountingHole:MountingHole_2.2mm_M2_Pad" (layer "F.Cu")
     (at 379.6 193.4)
     (descr "Mounting Hole 2.2mm, M2")
@@
   )
   (footprint "MountingHole:MountingHole_2.2mm_M2_Pad" (layer "F.Cu")
-    (at 212.2 116)
-    (descr "Mounting Hole 2.2mm, M2")
-    (tags "mounting hole 2.2mm m2")
-    (property "Sheetfile" "BackPCB-Acry.kicad_sch")
-    (property "Sheetname" "")
-    (attr exclude_from_pos_files)
-    (fp_text reference "H6" (at 0 -3.2) (layer "Dwgs.User")
-      (effects (font (size 1 1) (thickness 0.15)))
-    )
-    (fp_text value "MountingHole" (at 0 3.2) (layer "F.Fab")
-      (effects (font (size 1 1) (thickness 0.15)))
-    )
-    (fp_text user "${REFERENCE}" (at 0.3 0) (layer "F.Fab")
-      (effects (font (size 1 1) (thickness 0.15)))
-    )
-    (fp_circle (center 0 0) (end 2.2 0) (layer "Cmts.User") (width 0.1) (fill none))
-    (fp_circle (center 0 0) (end 2.45 0) (layer "F.CrtYd") (width 0.1) (fill none))
-    (pad "1" thru_hole circle locked (at 0 0) (size 4.4 4.4) (drill 2.2) (layers *.Cu *.Mask))
-  )
-  (footprint "MountingHole:MountingHole_2.2mm_M2_Pad" (layer "F.Cu")
-    (at 377.8 62.7)
-    (descr "Mounting Hole 2.2mm, M2")
-    (tags "mounting hole 2.2mm m2")
-    (property "Sheetfile" "BackPCB-Acry.kicad_sch")
-    (property "Sheetname" "")
-    (attr exclude_from_pos_files)
-    (fp_text reference "H1" (at 0 -3.2) (layer "Dwgs.User")
-      (effects (font (size 1 1) (thickness 0.15)))
-    )
-    (fp_text value "MountingHole" (at 0 3.2) (layer "F.Fab")
-      (effects (font (size 1 1) (thickness 0.15)))
-    )
-    (fp_text user "${REFERENCE}" (at 0.3 0) (layer "F.Fab")
-      (effects (font (size 1 1) (thickness 0.15)))
-    )
-    (fp_circle (center 0 0) (end 2.2 0) (layer "Cmts.User") (width 0.1) (fill none))
-    (fp_circle (center 0 0) (end 2.45 0) (layer "F.CrtYd") (width 0.1) (fill none))
-    (pad "1" thru_hole circle locked (at 0 0) (size 4.4 4.4) (drill 2.2) (layers *.Cu *.Mask))
-  )
-  (footprint "MountingHole:MountingHole_2.2mm_M2_Pad" (layer "F.Cu")
-    (at 40.1 196.3)
-    (descr "Mounting Hole 2.2mm, M2")
-    (tags "mounting hole 2.2mm m2")
-    (property "Sheetfile" "BackPCB-Acry.kicad_sch")
-    (property "Sheetname" "")
-    (attr exclude_from_pos_files)
-    (fp_text reference "H3" (at 0 -3.2) (layer "Dwgs.User")
-      (effects (font (size 1 1) (thickness 0.15)))
-    )
-    (fp_text value "MountingHole" (at 0 3.2) (layer "F.Fab")
-      (effects (font (size 1 1) (thickness 0.15)))
-    )
-    (fp_text user "${REFERENCE}" (at 0.3 0) (layer "F.Fab")
-      (effects (font (size 1 1) (thickness 0.15)))
-    )
-    (fp_circle (center 0 0) (end 2.2 0) (layer "Cmts.User") (width 0.1) (fill none))
-    (fp_circle (center 0 0) (end 2.45 0) (layer "F.CrtYd") (width 0.1) (fill none))
-    (pad "1" thru_hole circle locked (at 0 0) (size 4.4 4.4) (drill 2.2) (layers *.Cu *.Mask))
-  )
-  (footprint "MountingHole:MountingHole_2.2mm_M2_Pad" (layer "F.Cu")
-    (at 41.2 63.4)
-    (descr "Mounting Hole 2.2mm, M2")
-    (tags "mounting hole 2.2mm m2")
-    (property "Sheetfile" "BackPCB-Acry.kicad_sch")
-    (property "Sheetname" "")
-    (attr exclude_from_pos_files)
-    (fp_text reference "H0" (at 0 -3.2) (layer "Dwgs.User")
-      (effects (font (size 1 1) (thickness 0.15)))
-    )
-    (fp_text value "MountingHole" (at 0 3.2) (layer "F.Fab")
-      (effects (font (size 1 1) (thickness 0.15)))
-    )
-    (fp_text user "${REFERENCE}" (at 0.3 0) (layer "F.Fab")
-      (effects (font (size 1 1) (thickness 0.15)))
-    )
-    (fp_circle (center 0 0) (end 2.2 0) (layer "Cmts.User") (width 0.1) (fill none))
-    (fp_circle (center 0 0) (end 2.45 0) (layer "F.CrtYd") (width 0.1) (fill none))
-    (pad "1" thru_hole circle locked (at 0 0) (size 4.4 4.4) (drill 2.2) (layers *.Cu *.Mask))
-  )
-  (footprint "MountingHole:MountingHole_2.2mm_M2_Pad" (layer "F.Cu")
     (at 48.3 116)
     (descr "Mounting Hole 2.2mm, M2")
@@
   )
   (footprint "MountingHole:MountingHole_2.2mm_M2_Pad" (layer "F.Cu")
-    (at 48.3 116)
-    (descr "Mounting Hole 2.2mm, M2")
-    (tags "mounting hole 2.2mm m2")
-    (property "Sheetfile" "BackPCB-Acry.kicad_sch")
-    (property "Sheetname" "")
-    (attr exclude_from_pos_files)
-    (fp_text reference "H9" (at 0 -3.2) (layer "F.Fab")
-      (effects (font (size 1 1) (thickness 0.15)))
-    )
-    (fp_text value "MountingHole" (at 0 3.2) (layer "B.Fab")
-      (effects (font (size 1 1) (thickness 0.15)))
-    )
-    (fp_text user "${REFERENCE}" (at 0.3 0) (layer "F.Fab")
-      (effects (font (size 1 1) (thickness 0.15)))
-    )
-    (fp_circle (center 0 0) (end 2.2 0) (layer "Cmts.User") (width 0.1) (fill none))
-    (fp_circle (center 0 0) (end 2.45 0) (layer "F.CrtYd") (width 0.1) (fill none))
-    (pad "1" thru_hole circle locked (at 0 0) (size 4.4 4.4) (drill 2.2) (layers *.Cu *.Mask))
-  )
-  (footprint "MountingHole:MountingHole_2.2mm_M2_Pad" (layer "F.Cu")
     (at 376 116)
     (descr "Mounting Hole 2.2mm, M2")
@@
   )
   (footprint "MountingHole:MountingHole_2.2mm_M2_Pad" (layer "F.Cu")
-    (at 325.2 209.9)
+    (at 325.2 209.85)
     (descr "Mounting Hole 2.2mm, M2")
     (tags "mounting hole 2.2mm m2")
@@
   )
   (footprint "MountingHole:MountingHole_2.2mm_M2_Pad" (layer "F.Cu")
-    (at 182.9 63.4)
+    (at 182.9 63.75)
     (descr "Mounting Hole 2.2mm, M2")
     (tags "mounting hole 2.2mm m2")
@@
   )
   (footprint "MountingHole:MountingHole_2.2mm_M2_Pad" (layer "F.Cu")
-    (at 40.1 196.3)
+    (at 40.2 197)
     (descr "Mounting Hole 2.2mm, M2")
     (tags "mounting hole 2.2mm m2")
@@
   )
   (footprint "MountingHole:MountingHole_2.2mm_M2_Pad" (layer "F.Cu")
-    (at 203.9 176)
+    (at 203.85 177.3)
     (descr "Mounting Hole 2.2mm, M2")
     (tags "mounting hole 2.2mm m2")
@@
   )
   (footprint "MountingHole:MountingHole_2.2mm_M2_Pad" (layer "F.Cu")
-    (at 377.8 62.7)
+    (at 379.8 63.4)
     (descr "Mounting Hole 2.2mm, M2")
     (tags "mounting hole 2.2mm m2")
@@
   (gr_line (start 380.767 215.785) (end 39.767 215.785) (layer "Edge.Cuts") (width 0.1))
   (gr_arc (start 380.767 59.485) (mid 382.88832 60.36368) (end 383.767 62.485) (layer "Edge.Cuts") (width 0.1))
-  (gr_text "<Stepped\nNotStepped>" (at 52.7 171.8) (layer "F.Cu")
-    (effects (font (size 0.8 0.8) (thickness 0.15)))
-  )
   (gr_text "http://mechboards.co.uk" (at 210.27 148.49) (layer "F.Cu")
     (effects (font (size 2 2) (thickness 0.5)))
@@
     (connect_pads (clearance 0))
     (min_thickness 0.254)
-    (keepout (tracks not_allowed) (vias not_allowed) (pads not_allowed ) (copperpour not_allowed) (footprints not_allowed))
+    (keepout (tracks not_allowed) (vias not_allowed) (pads not_allowed) (copperpour not_allowed) (footprints not_allowed))
     (fill (thermal_gap 0.508) (thermal_bridge_width 0.508))
     (polygon
@@
     (connect_pads (clearance 0))
     (min_thickness 0.254)
-    (keepout (tracks not_allowed) (vias not_allowed) (pads not_allowed ) (copperpour not_allowed) (footprints not_allowed))
+    (keepout (tracks not_allowed) (vias not_allowed) (pads not_allowed) (copperpour not_allowed) (footprints not_allowed))
     (fill (thermal_gap 0.508) (thermal_bridge_width 0.508))
     (polygon
