File: KICAD PCBs/FrontPCB-Acrylic/FrontPCB.kicad_pcb (KiCad board)
At the start: 2 copper layers, 347 x 123.8 mm, 15 parts

Commit message: another small correction
Other:
- board text removed: "https://github.com/Envious-Data/Env-KB"
Changed lines of the file:
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@@
   (gr_arc (start 234.6625 155.825) (mid 234.516053 156.178553) (end 234.1625 156.325) (layer "Edge.Cuts") (width 0.1))
   (gr_arc (start 173.5375 137.275) (mid 173.183947 137.128553) (end 173.0375 136.775) (layer "Edge.Cuts") (width 0.1))
-  (gr_text "https://github.com/Envious-Data/Env-KB" (at 256.225 74.735) (layer "Eco2.User")
-    (effects (font (size 1 1) (thickness 0.2)) (justify right mirror))
-  )
   (gr_text "PLEASE CHECK ALIGNMENT OF \"HRO-TYPE-C-31-M-12\"" (at 212.225 52.535) (layer "F.Fab")
     (effects (font (size 1 1) (thickness 0.15)))

Commit message: Adjusted to fit JLCPCBs minimum width requirement, Generated Gerbers and DXF for top cover.
Other:
- board size 347 x 123.8 mm -> 350.6 x 126.8 mm

Commit message: modified switch plate and backplate
Parts:
- removed the H10 at (376.0, 116.0) (x2)
- removed the H3 at (40.1, 196.3) (x2)
- removed the H6 at (212.2, 116.0) (x2)
- removed the H9 at (48.3, 116.0) (x2)
- added H10: MountingHole, MountingHole:MountingHole_2.2mm_M2_Pad, F.Cu at (376.1, 116.2)
- added H3: MountingHole, MountingHole:MountingHole_2.2mm_M2_Pad, F.Cu at (40.3, 197.2)
- added H4: MountingHole, MountingHole:MountingHole_2.2mm_M2_Pad, F.Cu at (379.7, 193.6)
- added H4: MountingHole, MountingHole:MountingHole_2.2mm_M2_Pad, F.Cu at (325.3, 210.1)
- added H6: MountingHole, MountingHole:MountingHole_2.2mm_M2_Pad, F.Cu at (212.3, 116.2)
- added H9: MountingHole, MountingHole:MountingHole_2.2mm_M2_Pad, F.Cu at (48.4, 116.2)
- moved H7 1.50 mm to (203.9, 177.5)
