File: KICAD PCBs/MainPCB/ENV_KB.kicad_pcb (KiCad board)
At the start: 2 copper layers, 347 x 156.3 mm, 238 parts

Commit message: Modified mount holes for MBUK part inventory
Parts:
- H0 (x2), H1 (x2), H10 (x2), H11, H3 (x2), H4 (x2), H6 (x2), H7, H9 (x2): footprint MountingHole:MountingHole_2.2mm_M2_Pad -> MountingHole:MountingHole_3.5mm
Routing:
- net row5: track 344.6 -> 345.7 mm
- net GND: track 67.6 -> 68.5 mm

Commit message: Modified board to fit future plans
Parts:
- removed the H0 at (41.2, 63.4)
- removed the H1 at (377.8, 62.7)
- removed the H10 at (376.0, 116.0)
- removed the H3 at (40.1, 196.3)
- removed the H6 at (212.2, 116.0)
- removed the H9 at (48.3, 116.0)
- removed the K_0 at (46.7, 101.7)
- removed kibuzzard-628AE860: G***, kibuzzard-628AE860
- removed kibuzzard-628AE868: G***, kibuzzard-628AE868
- removed kibuzzard-628AE874: G***, kibuzzard-628AE874
- removed kibuzzard-628AE882: G***, kibuzzard-628AE882
- removed kibuzzard-628AE8A6: G***, kibuzzard-628AE8A6
- removed kibuzzard-628AE933: G***, kibuzzard-628AE933
- removed kibuzzard-628AE966: G***, kibuzzard-628AE966
- added kibuzzard-6376D46A (x2): G***, kibuzzard-6376D46A, F.Cu at (375.6, 172.3)
- D0, D1, D10, D11, D12, D13, D14, D15, D16, D17, D18, D19, D2, D20, D21, D22, D23, D24, D25, D26, D27, D28, D29, D29BS2, D3, D30, D31, D32, D33, D34, D35, D36, D37, D38, D39, D4, D40, D41, D42, D43, D44, D45, D46, D47, D48, D49, D5, D50, D51, D52, D53, D54, D55, D56, D57, D58, D59, D6, D60, D61, D62, D63, D64, D65, D66, D67, D68, D69, D7, D70, D71, D72, D73, D74, D75, D76, D77, D78, D79, D8, D80, D81, D81A1, D81A2, D82, D83, D84, D85, D86, D87, D88, D89, D9: footprint Diode_THT:D_DO-35_SOD27_P7.62mm_Horizontal -> EnvExtras:DiodeCustomSMDTHT
- moved D88 4.00 mm to (381.7, 70.6)
- moved H1 2.12 mm to (379.8, 63.4)
- moved H7 1.30 mm to (203.8, 177.3)
- moved H3 0.71 mm to (40.2, 197.0)
- moved H11 0.35 mm to (182.9, 63.8)
Routing:
- net row2: track 366.9 -> 480.7 mm
- net row0: track 371.5 -> 475.6 mm
- net row3: track 361.8 -> 457.8 mm
- net row5: track 345.7 -> 409.5 mm
- net row4: track 320.1 -> 378.2 mm
- net row6: track 363.1 -> 406.3 mm
- net Net-(D86-Pad2): track 165.3 -> 182.5 mm, vias 0 -> 4
- net col0: track 338.8 -> 345.0 mm
- net Net-(D0-Pad2): track 12.1 -> 14.7 mm, vias 0 -> 1
- net Net-(D33-Pad2): track 70.9 -> 68.5 mm
- net Net-(D16-Pad2): track 49.2 -> 51.3 mm
- net Resetbtn: track 62.7 -> 61.0 mm
- net Net-(D88-Pad2): track 226.4 -> 224.8 mm
- net col14: track 191.5 -> 190.7 mm
- net Net-(D78-Pad2): track 146.8 -> 147.6 mm
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Other:
- board text added: "Fit Switch here for ISO Enter"
- board text added: "Original Variant: https://github.com/Envious-Data/Env-KB MBUK Modified Ver: https://github.com/mechboardsguides/Env-KB-MBUK"
- board text removed: "https://github.com/Envious-Data/Env-KB"

Commit message: updated mount holes to be correct
Parts:
- D89: footprint EnvExtras:DiodeCustomSMDTHT -> Diode_THT:D_DO-35_SOD27_P7.62mm_Horizontal
- renumbered H4 to H5
