File: KICAD PCBs/MainPCB/ENV_KB.kicad_sch (KiCad schematic)
At the start: 211 parts

Commit message: Modified mount holes for MBUK part inventory
Parts:
- H0, H1, H10, H11, H3, H4, H6, H7, H9: footprint MountingHole:MountingHole_2.2mm_M2_Pad -> MountingHole:MountingHole_3.5mm
Changed lines of the file:
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@@
       (effects (font (size 1.27 1.27)) (justify left))
     )
-    (property "Footprint" "MountingHole:MountingHole_2.2mm_M2_Pad" (id 2) (at 167.64 240.03 0)
+    (property "Footprint" "MountingHole:MountingHole_3.5mm" (id 2) (at 167.64 240.03 0)
       (effects (font (size 1.27 1.27)) hide)
     )
@@
       (effects (font (size 1.27 1.27)) (justify left))
     )
-    (property "Footprint" "MountingHole:MountingHole_2.2mm_M2_Pad" (id 2) (at 167.64 224.79 0)
+    (property "Footprint" "MountingHole:MountingHole_3.5mm" (id 2) (at 167.64 224.79 0)
       (effects (font (size 1.27 1.27)) hide)
     )
@@
       (effects (font (size 1.27 1.27)) (justify left))
     )
-    (property "Footprint" "MountingHole:MountingHole_2.2mm_M2_Pad" (id 2) (at 167.64 229.87 0)
+    (property "Footprint" "MountingHole:MountingHole_3.5mm" (id 2) (at 167.64 229.87 0)
       (effects (font (size 1.27 1.27)) hide)
     )
@@
       (effects (font (size 1.27 1.27)) (justify left))
     )
-    (property "Footprint" "MountingHole:MountingHole_2.2mm_M2_Pad" (id 2) (at 167.64 245.11 0)
+    (property "Footprint" "MountingHole:MountingHole_3.5mm" (id 2) (at 167.64 245.11 0)
       (effects (font (size 1.27 1.27)) hide)
     )
@@
       (effects (font (size 1.27 1.27)) (justify left))
     )
-    (property "Footprint" "MountingHole:MountingHole_2.2mm_M2_Pad" (id 2) (at 167.64 270.51 0)
+    (property "Footprint" "MountingHole:MountingHole_3.5mm" (id 2) (at 167.64 270.51 0)
       (effects (font (size 1.27 1.27)) hide)
     )
@@
       (effects (font (size 1.27 1.27)) (justify left))
     )
-    (property "Footprint" "MountingHole:MountingHole_2.2mm_M2_Pad" (id 2) (at 167.64 275.59 0)
+    (property "Footprint" "MountingHole:MountingHole_3.5mm" (id 2) (at 167.64 275.59 0)
       (effects (font (size 1.27 1.27)) hide)
     )
@@
       (effects (font (size 1.27 1.27)) (justify left))
     )
-    (property "Footprint" "MountingHole:MountingHole_2.2mm_M2_Pad" (id 2) (at 167.64 255.27 0)
+    (property "Footprint" "MountingHole:MountingHole_3.5mm" (id 2) (at 167.64 255.27 0)
       (effects (font (size 1.27 1.27)) hide)
     )
@@
       (effects (font (size 1.27 1.27)) (justify left))
     )
-    (property "Footprint" "MountingHole:MountingHole_2.2mm_M2_Pad" (id 2) (at 167.64 260.35 0)
+    (property "Footprint" "MountingHole:MountingHole_3.5mm" (id 2) (at 167.64 260.35 0)
       (effects (font (size 1.27 1.27)) hide)
     )
@@
       (effects (font (size 1.27 1.27)) (justify left))
     )
-    (property "Footprint" "MountingHole:MountingHole_2.2mm_M2_Pad" (id 2) (at 167.64 265.43 0)
+    (property "Footprint" "MountingHole:MountingHole_3.5mm" (id 2) (at 167.64 265.43 0)
       (effects (font (size 1.27 1.27)) hide)
     )
@@
     )
     (path "/00000000-0000-0000-0000-0000605938c3"
-      (reference "H0") (unit 1) (value "MountingHole") (footprint "MountingHole:MountingHole_2.2mm_M2_Pad")
+      (reference "H0") (unit 1) (value "MountingHole") (footprint "MountingHole:MountingHole_3.5mm")
     )
     (path "/00000000-0000-0000-0000-0000605bd366"
-      (reference "H1") (unit 1) (value "MountingHole") (footprint "MountingHole:MountingHole_2.2mm_M2_Pad")
+      (reference "H1") (unit 1) (value "MountingHole") (footprint "MountingHole:MountingHole_3.5mm")
     )
     (path "/00000000-0000-0000-0000-00006058bc08"
-      (reference "H3") (unit 1) (value "MountingHole") (footprint "MountingHole:MountingHole_2.2mm_M2_Pad")
+      (reference "H3") (unit 1) (value "MountingHole") (footprint "MountingHole:MountingHole_3.5mm")
     )
     (path "/00000000-0000-0000-0000-00006068a680"
-      (reference "H4") (unit 1) (value "MountingHole") (footprint "MountingHole:MountingHole_2.2mm_M2_Pad")
+      (reference "H4") (unit 1) (value "MountingHole") (footprint "MountingHole:MountingHole_3.5mm")
     )
     (path "/00000000-0000-0000-0000-000060748b43"
-      (reference "H6") (unit 1) (value "MountingHole") (footprint "MountingHole:MountingHole_2.2mm_M2_Pad")
+      (reference "H6") (unit 1) (value "MountingHole") (footprint "MountingHole:MountingHole_3.5mm")
     )
     (path "/00000000-0000-0000-0000-00006077360a"
-      (reference "H7") (unit 1) (value "MountingHole") (footprint "MountingHole:MountingHole_2.2mm_M2_Pad")
+      (reference "H7") (unit 1) (value "MountingHole") (footprint "MountingHole:MountingHole_3.5mm")
     )
     (path "/00000000-0000-0000-0000-000060717f95"
-      (reference "H9") (unit 1) (value "MountingHole") (footprint "MountingHole:MountingHole_2.2mm_M2_Pad")
+      (reference "H9") (unit 1) (value "MountingHole") (footprint "MountingHole:MountingHole_3.5mm")
     )
     (path "/00000000-0000-0000-0000-0000607429b3"
-      (reference "H10") (unit 1) (value "MountingHole") (footprint "MountingHole:MountingHole_2.2mm_M2_Pad")
+      (reference "H10") (unit 1) (value "MountingHole") (footprint "MountingHole:MountingHole_3.5mm")
     )
     (path "/0eca823b-b704-4c12-9f7b-5d1293eeb888"
-      (reference "H11") (unit 1) (value "MountingHole") (footprint "MountingHole:MountingHole_2.2mm_M2_Pad")
+      (reference "H11") (unit 1) (value "MountingHole") (footprint "MountingHole:MountingHole_3.5mm")
     )
     (path "/00000000-0000-0000-0000-0000605cd72c"

Commit message: Modified board to fit future plans
Parts:
- D0, D1, D10, D11, D12, D13, D14, D15, D16, D17, D18, D19, D2, D20, D21, D22, D23, D24, D25, D26, D27, D28, D29, D29BS2, D3, D30, D31, D32, D33, D34, D35, D36, D37, D38, D39, D4, D40, D41, D42, D43, D44, D45, D46, D47, D48, D49, D5, D50, D51, D52, D53, D54, D55, D56, D57, D58, D59, D6, D60, D61, D62, D63, D64, D65, D66, D67, D68, D69, D7, D70, D71, D72, D73, D74, D75, D76, D77, D78, D79, D8, D80, D81, D81A1, D81A2, D82, D83, D84, D85, D86, D87, D88, D9: footprint Diode_THT:D_DO-35_SOD27_P7.62mm_Horizontal -> EnvExtras:DiodeCustomSMDTHT

Commit message: updated mount holes to be correct
Parts:
- added H5: MountingHole, MountingHole:MountingHole_3.5mm, symbol Mechanical:MountingHole
Changed lines of the file:
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@@
     (pin "2")
+  )
+  (symbol (lib_id "Mechanical:MountingHole") (at 167.64 249.555 0) (unit 1)
+    (in_bom yes) (on_board yes)
+    (property "Reference" "H5" (id 0) (at 170.18 248.3866 0)
+      (effects (font (size 1.27 1.27)) (justify left))
+    )
+    (property "Value" "MountingHole" (id 1) (at 170.18 250.698 0)
+      (effects (font (size 1.27 1.27)) (justify left))
+    )
+    (property "Footprint" "MountingHole:MountingHole_3.5mm" (id 2) (at 167.64 249.555 0)
+      (effects (font (size 1.27 1.27)) hide)
+    )
+    (property "Datasheet" "~" (id 3) (at 167.64 249.555 0)
+      (effects (font (size 1.27 1.27)) hide)
+    )
   )
   (symbol (lib_id "Device:D_Small") (at 212.09 185.42 90) (unit 1)
@@
       (reference "H4") (unit 1) (value "MountingHole") (footprint "MountingHole:MountingHole_3.5mm")
     )
+    (path "/7ded76f3-1df2-4d26-b7a3-0ed8a6f3e4b3"
+      (reference "H5") (unit 1) (value "MountingHole") (footprint "MountingHole:MountingHole_3.5mm")
+    )
     (path "/00000000-0000-0000-0000-000060748b43"
