File: KICAD PCBs/MainPCB_HS/EnvKB_HS.kicad_sch (KiCad schematic)
At the start: 209 parts

Commit message: Modified mount holes for MBUK part inventory
Parts:
- H0, H1, H10, H2, H3, H4, H5, H6, H7, H9: footprint MountingHole:MountingHole_2.2mm_M2_Pad -> MountingHole:MountingHole_3.5mm
Changed lines of the file:
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@@
       (effects (font (size 1.27 1.27)) (justify left))
     )
-    (property "Footprint" "MountingHole:MountingHole_2.2mm_M2_Pad" (id 2) (at 147.32 270.51 0)
+    (property "Footprint" "MountingHole:MountingHole_3.5mm" (id 2) (at 147.32 270.51 0)
       (effects (font (size 1.27 1.27)) hide)
     )
@@
       (effects (font (size 1.27 1.27)) (justify left))
     )
-    (property "Footprint" "MountingHole:MountingHole_2.2mm_M2_Pad" (id 2) (at 137.16 270.51 0)
+    (property "Footprint" "MountingHole:MountingHole_3.5mm" (id 2) (at 137.16 270.51 0)
       (effects (font (size 1.27 1.27)) hide)
     )
@@
       (effects (font (size 1.27 1.27)) (justify left))
     )
-    (property "Footprint" "MountingHole:MountingHole_2.2mm_M2_Pad" (id 2) (at 142.24 270.51 0)
+    (property "Footprint" "MountingHole:MountingHole_3.5mm" (id 2) (at 142.24 270.51 0)
       (effects (font (size 1.27 1.27)) hide)
     )
@@
       (effects (font (size 1.27 1.27)) (justify left))
     )
-    (property "Footprint" "MountingHole:MountingHole_2.2mm_M2_Pad" (id 2) (at 152.4 270.51 0)
+    (property "Footprint" "MountingHole:MountingHole_3.5mm" (id 2) (at 152.4 270.51 0)
       (effects (font (size 1.27 1.27)) hide)
     )
@@
       (effects (font (size 1.27 1.27)) (justify left))
     )
-    (property "Footprint" "MountingHole:MountingHole_2.2mm_M2_Pad" (id 2) (at 167.64 270.51 0)
+    (property "Footprint" "MountingHole:MountingHole_3.5mm" (id 2) (at 167.64 270.51 0)
       (effects (font (size 1.27 1.27)) hide)
     )
@@
       (effects (font (size 1.27 1.27)) (justify left))
     )
-    (property "Footprint" "MountingHole:MountingHole_2.2mm_M2_Pad" (id 2) (at 172.72 270.51 0)
+    (property "Footprint" "MountingHole:MountingHole_3.5mm" (id 2) (at 172.72 270.51 0)
       (effects (font (size 1.27 1.27)) hide)
     )
@@
       (effects (font (size 1.27 1.27)) (justify left))
     )
-    (property "Footprint" "MountingHole:MountingHole_2.2mm_M2_Pad" (id 2) (at 157.48 270.51 0)
+    (property "Footprint" "MountingHole:MountingHole_3.5mm" (id 2) (at 157.48 270.51 0)
       (effects (font (size 1.27 1.27)) hide)
     )
@@
       (effects (font (size 1.27 1.27)) (justify left))
     )
-    (property "Footprint" "MountingHole:MountingHole_2.2mm_M2_Pad" (id 2) (at 162.56 270.51 0)
+    (property "Footprint" "MountingHole:MountingHole_3.5mm" (id 2) (at 162.56 270.51 0)
       (effects (font (size 1.27 1.27)) hide)
     )
@@
       (effects (font (size 1.27 1.27)) (justify left))
     )
-    (property "Footprint" "MountingHole:MountingHole_2.2mm_M2_Pad" (id 2) (at 132.08 270.51 0)
+    (property "Footprint" "MountingHole:MountingHole_3.5mm" (id 2) (at 132.08 270.51 0)
       (effects (font (size 1.27 1.27)) hide)
     )
@@
       (effects (font (size 1.27 1.27)) (justify left))
     )
-    (property "Footprint" "MountingHole:MountingHole_2.2mm_M2_Pad" (id 2) (at 127 270.51 0)
+    (property "Footprint" "MountingHole:MountingHole_3.5mm" (id 2) (at 127 270.51 0)
       (effects (font (size 1.27 1.27)) hide)
     )
@@
     )
     (path "/00000000-0000-0000-0000-0000605938c3"
-      (reference "H0") (unit 1) (value "MountingHole") (footprint "MountingHole:MountingHole_2.2mm_M2_Pad")
+      (reference "H0") (unit 1) (value "MountingHole") (footprint "MountingHole:MountingHole_3.5mm")
     )
     (path "/00000000-0000-0000-0000-0000605bd366"
-      (reference "H1") (unit 1) (value "MountingHole") (footprint "MountingHole:MountingHole_2.2mm_M2_Pad")
+      (reference "H1") (unit 1) (value "MountingHole") (footprint "MountingHole:MountingHole_3.5mm")
     )
     (path "/00000000-0000-0000-0000-000061411d60"
-      (reference "H2") (unit 1) (value "MountingHole") (footprint "MountingHole:MountingHole_2.2mm_M2_Pad")
+      (reference "H2") (unit 1) (value "MountingHole") (footprint "MountingHole:MountingHole_3.5mm")
     )
     (path "/00000000-0000-0000-0000-00006058bc08"
-      (reference "H3") (unit 1) (value "MountingHole") (footprint "MountingHole:MountingHole_2.2mm_M2_Pad")
+      (reference "H3") (unit 1) (value "MountingHole") (footprint "MountingHole:MountingHole_3.5mm")
     )
     (path "/00000000-0000-0000-0000-00006068a680"
-      (reference "H4") (unit 1) (value "MountingHole") (footprint "MountingHole:MountingHole_2.2mm_M2_Pad")
+      (reference "H4") (unit 1) (value "MountingHole") (footprint "MountingHole:MountingHole_3.5mm")
     )
     (path "/00000000-0000-0000-0000-00006162a1bf"
-      (reference "H5") (unit 1) (value "MountingHole") (footprint "MountingHole:MountingHole_2.2mm_M2_Pad")
+      (reference "H5") (unit 1) (value "MountingHole") (footprint "MountingHole:MountingHole_3.5mm")
     )
     (path "/00000000-0000-0000-0000-000060748b43"
-      (reference "H6") (unit 1) (value "MountingHole") (footprint "MountingHole:MountingHole_2.2mm_M2_Pad")
+      (reference "H6") (unit 1) (value "MountingHole") (footprint "MountingHole:MountingHole_3.5mm")
     )
     (path "/00000000-0000-0000-0000-00006077360a"
-      (reference "H7") (unit 1) (value "MountingHole") (footprint "MountingHole:MountingHole_2.2mm_M2_Pad")
+      (reference "H7") (unit 1) (value "MountingHole") (footprint "MountingHole:MountingHole_3.5mm")
     )
     (path "/00000000-0000-0000-0000-000060717f95"
-      (reference "H9") (unit 1) (value "MountingHole") (footprint "MountingHole:MountingHole_2.2mm_M2_Pad")
+      (reference "H9") (unit 1) (value "MountingHole") (footprint "MountingHole:MountingHole_3.5mm")
     )
     (path "/00000000-0000-0000-0000-0000607429b3"
-      (reference "H10") (unit 1) (value "MountingHole") (footprint "MountingHole:MountingHole_2.2mm_M2_Pad")
+      (reference "H10") (unit 1) (value "MountingHole") (footprint "MountingHole:MountingHole_3.5mm")
     )
     (path "/00000000-0000-0000-0000-0000603522c8"

Commit message: Overhauled HS version so there is design parity
Parts:
- removed H2, H5: MountingHole, MountingHole:MountingHole_3.5mm, symbol Mechanical:MountingHole_Pad
- removed LEDRESISTOR2: 5.1K Resistor 0805, Resistor_SMD:R_0805_2012Metric_Pad1.20x1.40mm_HandSolder, symbol Device:R_Small
- removed PowerLED1: LED 0805, LED_SMD:LED_0805_2012Metric, symbol Device:LED
- removed RESISTOR2, RESISTOR3: 5.1kohm 0805, Resistor_SMD:R_0805_2012Metric, symbol Device:R_Small
- removed Stab1: Stabilizer, Mounting_Keyboard_Stabilizer:Stabilizer_Cherry_MX_6.25u, symbol Mechanical:MountingHole
- removed Stab2, Stab3, Stab4, Stab5, Stab6: Stabilizer, Mounting_Keyboard_Stabilizer:Stabilizer_Cherry_MX_2u, symbol Mechanical:MountingHole
- added D29BS2, D81A1, D81A2: D, EnvExtras:DiodeCustomSMDTHT, symbol Device:D_Small
- added H11: MountingHole, EnvExtras:SMDNUT-M2, symbol Mechanical:MountingHole
- added I2CHeader0: Conn_01x04, Connector_PinSocket_2.54mm:PinSocket_1x04_P2.54mm_Vertical, symbol Connector_Generic:Conn_01x04
- added K_29BS1, K_29BS2, K_81A1, K_81A2: KEYSW, MX_Only:MXOnly-1U-Hotswap-Modified, symbol MX_Alps_Hybrid:MX-NoLED
- added STAB1, STAB2, STAB3, STAB4, STAB5, STAB6, STAB7: Stabilizer, Mounting_Keyboard_Stabilizer:Stabilizer_Cherry_MX_2u, symbol Mechanical:MountingHole
- D0, D1, D10, D11, D12, D13, D14, D15, D16, D17, D18, D19, D2, D20, D21, D22, D23, D24, D25, D26, D27, D28, D29, D3, D30, D31, D32, D33, D34, D35, D36, D37, D38, D39, D4, D40, D41, D42, D43, D44, D45, D46, D47, D48, D49, D5, D50, D51, D52, D53, D54, D55, D56, D57, D58, D59, D6, D60, D61, D62, D63, D64, D65, D66, D67, D68, D69, D7, D70, D71, D72, D73, D74, D75, D76, D77, D78, D79, D8, D80, D81, D82, D83, D84, D85, D86, D87, D88, D9: footprint EM_Extras:SOD-123+D_DO-35_SOD27_P7.62mm_Horizontal -> EnvExtras:DiodeCustomSMDTHT
- D89: footprint Diode_THT:D_DO-41_SOD81_P7.62mm_Horizontal -> Diode_THT:D_DO-35_SOD27_P7.62mm_Horizontal
- H0, H1, H10, H3, H4, H6, H7, H9: footprint MountingHole:MountingHole_3.5mm -> EnvExtras:SMDNUT-M2; symbol Mechanical:MountingHole_Pad -> Mechanical:MountingHole
- K_0, K_1, K_10, K_11, K_12, K_13, K_14, K_15, K_16, K_17, K_18, K_19, K_2, K_20, K_21, K_22, K_23, K_24, K_25, K_26, K_27, K_28, K_29, K_3, K_30, K_31, K_32, K_33, K_34, K_35, K_36, K_37, K_38, K_39, K_4, K_40, K_41, K_42, K_43, K_44, K_45, K_46, K_47, K_48, K_49, K_5, K_50, K_50A1, K_51, K_52, K_53, K_54, K_55, K_56, K_57, K_58, K_59, K_6, K_60, K_61, K_62, K_63, K_63B1, K_64, K_64B1, K_65, K_66, K_67, K_68, K_69, K_7, K_70, K_71, K_72, K_73, K_74, K_75, K_76, K_77, K_78, K_79, K_8, K_80, K_81, K_82, K_83, K_84, K_85, K_86, K_87, K_88, K_9: LCSC C2803348 -> (none)
- PowerLED0: value LED 3MM -> LED 3mm; footprint LED_THT:LED_D3.0mm_FlatTop -> LED_THT:LED_D3.0mm
- PowerLedResistor0: renamed from LEDRESISTOR1; value 5.1K Resistor 1/4w -> 47K Resistor; footprint Resistor_THT:R_Axial_DIN0207_L6.3mm_D2.5mm_P10.16mm_Horizontal -> Resistor_THT:R_Axial_DIN0207_L6.3mm_D2.5mm_P7.62mm_Horizontal
- RESISTOR0: value 5.1kohm 1/4w -> 5.1k; footprint Resistor_THT:R_Axial_DIN0207_L6.3mm_D2.5mm_P10.16mm_Horizontal -> Resistor_THT:R_Axial_DIN0207_L6.3mm_D2.5mm_P7.62mm_Horizontal
- RESISTOR1: value 5.1kohm 1/4 -> 5.1k; footprint Resistor_THT:R_Axial_DIN0207_L6.3mm_D2.5mm_P10.16mm_Horizontal -> Resistor_THT:R_Axial_DIN0207_L6.3mm_D2.5mm_P7.62mm_Horizontal
- SW-RST0: footprint Button_Switch_SMD:Panasonic_EVQPUM_EVQPUD -> Button_Switch_SMD:Panasonic_EVQPUL_EVQPUC
- USB1: value TYPE-C-31-M-14 -> HRO-TYPE-C-31-M-12
Connections:
- net 3.3V: now also I2CHeader0.2 (Pin_2)
- net GND: now also I2CHeader0.1 (Pin_1); no longer H0.1, H1.1, H10.1, H3.1, H4.1, H6.1, H7.1, H9.1
- net col13: now also K_29BS2.1 (COL)
- net col14: now also K_29BS1.1 (COL)
- net col5: now also K_81A1.1 (COL)
- net col7: now also K_81A2.1 (COL)
- net row2: now also D29BS2.1 (K)
- net row6: now also D81A1.1 (K), D81A2.1 (K)
- net at D29.2 (A), K_29.2 (ROW): now also K_29BS1.2 (ROW)
- net I2CSCL: now reaches RPI0.2 (GPIO1)
- net I2CSCL: now also I2CHeader0.3 (Pin_3)
- net at RESISTOR1.2: now also USB1.A5 (CC1); no longer USB1.B5 (CC2)
- net at RESISTOR0.1: now also USB1.B5 (CC2); no longer USB1.A5 (CC1)
- net LEDPIN renamed I2CSDA
- net I2CSDA: now also I2CHeader0.4 (Pin_4)
- new net: D29BS2.2 (A), K_29BS2.2 (ROW)
- new net: D81A2.2 (A), K_81A2.2 (ROW)
- new net: D81A1.2 (A), K_81A1.2 (ROW)
Other:
- note added: "Stepped capslock"
- note removed: "Do not install both resistors"
- note removed: "This needs double checking"
- moved on the sheet: USB1

Commit message: updated mount holes to be correct
Parts:
- added H5: MountingHole, EnvExtras:SMDNUT-M2, symbol Mechanical:MountingHole
Changed lines of the file:
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@@
     (pin "2")
+  )
+  (symbol (lib_id "Mechanical:MountingHole") (at 167.64 249.555 0) (unit 1)
+    (in_bom yes) (on_board yes)
+    (property "Reference" "H5" (id 0) (at 170.18 248.3866 0)
+      (effects (font (size 1.27 1.27)) (justify left))
+    )
+    (property "Value" "MountingHole" (id 1) (at 170.18 250.698 0)
+      (effects (font (size 1.27 1.27)) (justify left))
+    )
+    (property "Footprint" "EnvExtras:SMDNUT-M2" (id 2) (at 167.64 249.555 0)
+      (effects (font (size 1.27 1.27)) hide)
+    )
+    (property "Datasheet" "~" (id 3) (at 167.64 249.555 0)
+      (effects (font (size 1.27 1.27)) hide)
+    )
   )
   (symbol (lib_id "Mechanical:MountingHole") (at 229.235 202.565 0) (unit 1)
@@
       (reference "H4") (unit 1) (value "MountingHole") (footprint "EnvExtras:SMDNUT-M2")
     )
+    (path "/ad0cbb1b-8e9b-4e36-8a5f-4bbb3e0cdf87"
+      (reference "H5") (unit 1) (value "MountingHole") (footprint "EnvExtras:SMDNUT-M2")
+    )
     (path "/00000000-0000-0000-0000-000060748b43"
